File: 2023/PCB/WinterDeco2023.kicad_pcb (KiCad board)
At the start: 2 copper layers, 124 x 126.4 mm, 42 parts, among them J1 CONN_ICSP_UART, Q1 IRLML6402, SW1 TOUCH_SENSOR, U1 PIC18F14 (SOP20/SSOP20)

Commit message: Fixed swapped rows and columns
Connections:
- net /COL4 renamed /ROW4
- net /COL5 renamed /ROW5
- DB11 pad 1: /COL1 -> /ROW1
- DB12 pad 1: /COL2 -> /ROW2
- DB13 pad 1: /COL3 -> /ROW3
- DB21 pad 1: /COL1 -> /ROW1
- DB22 pad 1: /COL2 -> /ROW2
- DB23 pad 1: /COL3 -> /ROW3
- DB31 pad 1: /COL1 -> /ROW1
- DB32 pad 1: /COL2 -> /ROW2
- DB33 pad 1: /COL3 -> /ROW3
- DF11 pad 2: /COL1 -> /ROW1
- DF12 pad 2: /COL2 -> /ROW2
- DF13 pad 2: /COL3 -> /ROW3
- DF21 pad 2: /COL1 -> /ROW1
- DF22 pad 2: /COL2 -> /ROW2
- DF23 pad 2: /COL3 -> /ROW3
- DF31 pad 2: /COL1 -> /ROW1
- DF32 pad 2: /COL2 -> /ROW2
- DF33 pad 2: /COL3 -> /ROW3
- R1 pad 2: /ROW1 -> /COL1
- R2 pad 2: /ROW2 -> /COL2
- R3 pad 2: /ROW3 -> /COL3
- U1 pad 14: /ROW3 -> /COL3
- U1 pad 15: /ROW2 -> /COL2
- U1 pad 16: /ROW1 -> /COL1
- U1 pad 5: /COL3 -> /ROW3
- U1 pad 6: /COL2 -> /ROW2
- U1 pad 7: /COL1 -> /ROW1
Routing:
- net /ROW3: track 10.4 -> 173.8 mm
- net /COL3: track 173.8 -> 10.4 mm
- net /ROW1: track 5.55 -> 119.8 mm
- net /COL1: track 119.8 -> 5.55 mm
- net /ROW2: track 7.88 -> 72.3 mm, vias 0 -> 2
- net /COL2: track 72.3 -> 7.88 mm, vias 2 -> 0
